File: fpga_page5.kicad_sch (KiCad schematic)
At the start: 24 parts, among them U1 XC7S75-1FGGA484C

Commit message: Uploading...
Changed lines of the file:
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@@
 		)
 	)
-	(global_label "GND"
-		(shape input)
-		(at 207.01 67.31 180)
+	(label "GND"
+		(at 187.96 50.8 180)
 		(fields_autoplaced yes)
 		(effects
@@
 				(size 1.27 1.27)
 			)
-			(justify right)
-		)
-		(property "Intersheetrefs" "${INTERSHEET_REFS}"
-			(at 200.1543 67.31 0)
-			(effects
-				(font
-					(size 1.27 1.27)
-				)
-				(justify right)
-				(hide yes)
-			)
+			(justify right bottom)
 		)
 	)
-	(global_label "GND"
-		(shape input)
-		(at 207.01 72.39 180)
+	(label "GND"
+		(at 139.7 85.09 180)
 		(fields_autoplaced yes)
 		(effects
@@
 				(size 1.27 1.27)
 			)
-			(justify right)
-		)
-		(property "Intersheetrefs" "${INTERSHEET_REFS}"
-			(at 200.1543 72.39 0)
-			(effects
-				(font
-					(size 1.27 1.27)
-				)
-				(justify right)
-				(hide yes)
-			)
+			(justify right bottom)
 		)
 	)
-	(global_label "GND"
-		(shape input)
-		(at 152.4 72.39 180)
+	(label "VCC3V3"
+		(at 187.96 43.18 180)
 		(fields_autoplaced yes)
 		(effects
@@
 				(size 1.27 1.27)
 			)
-			(justify right)
-		)
-		(property "Intersheetrefs" "${INTERSHEET_REFS}"
-			(at 145.5443 72.39 0)
-			(effects
-				(font
-					(size 1.27 1.27)
-				)
-				(justify right)
-				(hide yes)
-			)
+			(justify right bottom)
 		)
 	)
-	(global_label "DDRVCC"
-		(shape input)
-		(at 139.7 77.47 180)
+	(label "GND"
+		(at 207.01 67.31 180)
 		(fields_autoplaced yes)
 		(effects
@@
 				(size 1.27 1.27)
 			)
-			(justify right)
-		)
-		(property "Intersheetrefs" "${INTERSHEET_REFS}"
-			(at 129.2762 77.47 0)
-			(effects
-				(font
-					(size 1.27 1.27)
-				)
-				(justify right)
-				(hide yes)
-			)
+			(justify right bottom)
 		)
 	)
-	(global_label "VCC3V3"
-		(shape input)
-		(at 152.4 64.77 180)
+	(label "DDRVCC"
+		(at 139.7 77.47 180)
 		(fields_autoplaced yes)
 		(effects
@@
 				(size 1.27 1.27)
 			)
-			(justify right)
-		)
-		(property "Intersheetrefs" "${INTERSHEET_REFS}"
-			(at 142.2786 64.77 0)
-			(effects
-				(font
-					(size 1.27 1.27)
-				)
-				(justify right)
-				(hide yes)
-			)
+			(justify right bottom)
 		)
 	)
-	(global_label "VCC3V3"
-		(shape input)
-		(at 187.96 43.18 180)
+	(label "VCC3V3"
+		(at 156.21 53.34 180)
 		(fields_autoplaced yes)
 		(effects
@@
 				(size 1.27 1.27)
 			)
-			(justify right)
-		)
-		(property "Intersheetrefs" "${INTERSHEET_REFS}"
-			(at 177.8386 43.18 0)
-			(effects
-				(font
-					(size 1.27 1.27)
-				)
-				(justify right)
-				(hide yes)
-			)
+			(justify right bottom)
 		)
 	)
-	(global_label "GND"
-		(shape input)
+	(label "GND"
 		(at 156.21 60.96 180)
 		(fields_autoplaced yes)
@@
 				(size 1.27 1.27)
 			)
-			(justify right)
-		)
-		(property "Intersheetrefs" "${INTERSHEET_REFS}"
-			(at 149.3543 60.96 0)
-			(effects
-				(font
-					(size 1.27 1.27)
-				)
-				(justify right)
-				(hide yes)
-			)
+			(justify right bottom)
 		)
 	)
-	(global_label "VCC3V3"
-		(shape input)
-		(at 156.21 53.34 180)
+	(label "VCC3V3"
+		(at 152.4 64.77 180)
 		(fields_autoplaced yes)
 		(effects
@@
 				(size 1.27 1.27)
 			)
-			(justify right)
-		)
-		(property "Intersheetrefs" "${INTERSHEET_REFS}"
-			(at 146.0886 53.34 0)
-			(effects
-				(font
-					(size 1.27 1.27)
-				)
-				(justify right)
-				(hide yes)
-			)
+			(justify right bottom)
 		)
 	)
-	(global_label "GND"
-		(shape input)
-		(at 139.7 85.09 180)
+	(label "GND"
+		(at 207.01 72.39 180)
 		(fields_autoplaced yes)
 		(effects
@@
 				(size 1.27 1.27)
 			)
-			(justify right)
-		)
-		(property "Intersheetrefs" "${INTERSHEET_REFS}"
-			(at 132.8443 85.09 0)
-			(effects
-				(font
-					(size 1.27 1.27)
-				)
-				(justify right)
-				(hide yes)
-			)
+			(justify right bottom)
 		)
 	)
-	(global_label "GND"
-		(shape input)
-		(at 187.96 50.8 180)
+	(label "GND"
+		(at 152.4 72.39 180)
 		(fields_autoplaced yes)
 		(effects
@@
 				(size 1.27 1.27)
 			)
-			(justify right)
-		)
-		(property "Intersheetrefs" "${INTERSHEET_REFS}"
-			(at 181.1043 50.8 0)
-			(effects
-				(font
-					(size 1.27 1.27)
-				)
-				(justify right)
-				(hide yes)
-			)
+			(justify right bottom)
 		)
 	)
@@
 		(dnp no)
 		(property "Reference" "R171"
-			(at 209.804 70.612 90)
+			(at 212.598 70.612 90)
 			(effects
 				(font
@@
 		)
 		(property "Value" "0"
-			(at 207.772 73.914 90)
+			(at 207.772 70.612 90)
 			(effects
 				(font
@@
 		(dnp no)
 		(property "Reference" "R170"
-			(at 209.804 65.532 90)
+			(at 212.598 65.532 90)
 			(effects
 				(font
@@
 		)
 		(property "Value" "0"
-			(at 207.772 68.834 90)
+			(at 207.772 65.532 90)
 			(effects
 				(font
