File: ftdi.kicad_sch (KiCad schematic)
At the start: 1 part, among them U5 FT2232HQ-TRAY

Commit message: Uploading...
Parts:
- removed U5: FT2232HQ-TRAY, FT2232HQ-TRAY:QFN50P900X900X100-65N, symbol New_Library:FT2232HQ-TRAY
- added C13, C15, C25, C28, C36: 4.7UF,1206, Capacitor_SMD:C_1206_3216Metric, symbol Aardonyx-rescue:C_Small-aardonyx
- added C14, C24, C27, C30, C37, C38, C39, C40, C41, C42, C43, C44: 0.1UF,0402, Capacitor_SMD:C_0402_1005Metric, symbol Aardonyx-rescue:C_Small-aardonyx
- added C26, C29: 18PF,0402, Capacitor_SMD:C_0402_1005Metric, symbol Aardonyx-rescue:C_Small-aardonyx
- added D3, D4: CG0603MLC-12E, Diode_SMD:D_0603_1608Metric, symbol Aardonyx-rescue:D_BI-aardonyx
- added FB1, FB2: 47E,FB,0603, Capacitor_SMD:C_0603_1608Metric, symbol Aardonyx-rescue:Ferrite_Bead_Small-aardonyx
- added FB10, FB6, FB7, FB8, FB9: 600E,FB,0402, Inductor_SMD:L_0402_1005Metric, symbol Aardonyx-rescue:Ferrite_Bead_Small-aardonyx
- added J3: USB_B_6PIN, Connector_USB:USB_B_OST_USB-B1HSxx_Horizontal, symbol Aardonyx-rescue:USB_B_6PIN
- added J4: USB_OTG, Connector_USB:USB_Micro-B_Amphenol_10103594-0001LF_Horizontal, symbol Aardonyx-rescue:USB_OTG-aardonyx
- added J5, J7: Conn_1x3_M, Connector_PinHeader_2.54mm:PinHeader_1x03_P2.54mm_Vertical, symbol Aardonyx-rescue:Conn_1x3_M-aardonyx
- added J6: Conn_1x8, Connector_PinHeader_2.54mm:PinHeader_1x08_P2.54mm_Vertical, symbol Aardonyx-rescue:Conn_1x8-aardonyx
- added R10, R4, R9: 0E, 0402, Resistor_SMD:R_0402_1005Metric, symbol Aardonyx-rescue:R_US-aardonyx
- added R11: 4.7KE,0402, Resistor_SMD:R_0402_1005Metric, symbol Aardonyx-rescue:R_US-aardonyx
- added R12: 10KE,0402, Resistor_SMD:R_0402_1005Metric, symbol Aardonyx-rescue:R_US-aardonyx
- added R13, R14, R15, R16, R17, R18, R19, R20, R21, R22, R23, R24, R25, R26, R7: 1KE,0402, Resistor_SMD:R_0402_1005Metric, symbol Aardonyx-rescue:R_US-aardonyx
- added R5, R6: 22E,0402, Resistor_SMD:R_0402_1005Metric, symbol Aardonyx-rescue:R_US-aardonyx
- added R8: 12KE,0402, Resistor_SMD:R_0402_1005Metric, symbol Aardonyx-rescue:R_US-aardonyx
- added TP1, TP2, TP3: TestPoint, TestPoint:TestPoint_Pad_D1.0mm, symbol Aardonyx-rescue:TestPoint-aardonyx
- added U11: FT2232H, Package_QFP:LQFP-64_10x10mm_P0.5mm, symbol Aardonyx-rescue:FT2232H-aardonyx
- added U5: 93LC56BT-I_OT, Package_TO_SOT_SMD:SOT-23-6, symbol Aardonyx-rescue:93LC56BT-I_OT
- added Y3: 12MHz, Aardonyx:Crystal_SMD_ROHS_CSM_7XDN_HandSoldering, symbol Aardonyx-rescue:Crystal-aardonyx
Connections:
- new net: FB1.2, J4.6 (SHLD1)
- new net: C28.1, C30.1, FB9.1, U11.9 (VPLL)
- new net: C13.1, FB6.1, J3.1 (VBUS)
- new net: C36.1, C37.1, FB10.1, U11.4 (VPHY)
- new net: C15.1, FB7.1, J4.1 (VBUS)
- new net: TP2.1, U11.60 (~{PWREN})
- new net: C29.1, U11.3 (OSCO), Y3.2
- new net: C26.1, U11.2 (OSCI), Y3.1
- new net: R8.1, U11.6 (REF)
- new net: R10.1, U11.39 (BDBUS1)
- new net: TP3.1, U11.36 (~{SUSPEND})
- new net: FB2.1, J3.5 (SHLD1)
- new net: U11.61 (EEDATA), U5.1 (DO), U5.3 (DI)
- new net: U11.62 (EECLK), U5.4 (CLK)
- new net: U11.63 (EECS), U5.5 (CS)
- new net: R9.1, U11.38 (BDBUS0)
- new net D+: R5.1, U11.8 (DP)
- new net D-: R6.1, U11.7 (DM)
- new net FT_RESET: R4.2, R7.2, TP1.1, U11.14 (~{RESET})
- new net GNDA: FB8.1, U11.10 (AGND)
- new net GNDREF: C13.2, C14.2, C15.2, C24.1, C25.2, C26.2, C27.2, C28.2, C29.2, C30.2, C36.2, C37.2, C38.2, C39.2, C40.2, C41.2, C42.2, C43.2, C44.2, D3.2 (A2), D4.2 (A2), FB1.1, FB2.2, FB8.2, J3.4 (GND), J4.5 (GND), J6.8 (Pin_8), J7.3 (Pin_3), R12.2, R14.2, R16.2, R18.2, R20.2, R22.2, R24.2, R26.2, R8.2, U11.1 (GND), U11.11 (GND), U11.13 (TEST), U11.15 (GND), U11.25 (GND), U11.35 (GND), U11.47 (GND), U11.5 (GND), U11.51 (GND), U5.2 (GND)
- new net PWRSAV: R11.2, R12.1, U11.59 (BCBUS7)
- new net RESET: R4.1
- new net TCK: J6.2 (Pin_2), R13.2, R14.1, U11.16 (ADBUS0)
- new net TDI: J6.5 (Pin_5), R23.2, R24.1, U11.17 (ADBUS1)
- new net TDO: J6.6 (Pin_6), R25.2, R26.1, U11.18 (ADBUS2)
- new net TMS: J6.4 (Pin_4), R19.2, R20.1, U11.19 (ADBUS3)
- new net TRST: J6.3 (Pin_3), R15.2, R16.1, U11.22 (ADBUS5)
- new net UART0_RX: J7.1 (Pin_1), R17.2, R18.1, R9.2
- new net UART0_TX: J7.2 (Pin_2), R10.2, R21.2, R22.1
- new net USB_D+: D3.1 (A1), J3.3 (D+), J4.3 (D+), R5.2
- new net USB_D-: D4.1 (A1), J3.2 (D-), J4.2 (D-), R6.2
- new net V3P3: C14.1, C24.2, C41.1, C42.1, C43.1, C44.1, FB10.2, FB9.2, J6.1 (Pin_1), R13.1, R15.1, R17.1, R19.1, R21.1, R23.1, R25.1, R7.1, U11.20 (VCCIO), U11.31 (VCCIO), U11.42 (VCCIO), U11.50 (VREGIN), U11.56 (VCCIO), U5.6 (VCC)
- new net VBUS: J5.2 (Pin_2), R11.1
- new net VBUS_USB1: FB6.2, J5.1 (Pin_1)
- new net VBUS_USB2: FB7.2, J5.3 (Pin_3)
- new net VCORE_FTDI: C25.1, C27.1, C38.1, C39.1, C40.1, U11.12 (VCORE), U11.37 (VCORE), U11.49 (VREGOUT), U11.64 (VCORE)
- no-connect marks 0 -> 26
Other:
- note added: "2Kb 16bit Serial EEPROM"
- note added: "64PIN LQFP"
- note added: "SOT23-6"
- note added: "Short 1 & 2, VBUS = VBUS_USB1 Short 2 & 3, VBUS = VBUS_USB2"
- note added: "USB - JTAG/UART DUAL PORT CONVERTER"
- note added: "Use J1 for high loads"
- note added: "Use J17 for low power applications"
