File: power.kicad_sch (KiCad schematic)
At the start: 1 part, among them U2 ADP5052ACPZ-R7

Commit message: Uploading...
Parts:
- added D2: LED, symbol Device:LED
- added JP3, JP4: Conn_01x02, symbol Connector_Generic:Conn_01x02
- added R2, R3: 10m, symbol Device:R
Connections:
- net DDR1V35: now reaches U2.10 (SW4)
- net DDR1V35: now also U2.37 (EN1), U2.5 (EN5)
- net VCC1V8: now reaches U2.14 (EN4)
- net VCC5V0: now reaches U2.23 (EN2)
- net VCC5V0: now also U2.24 (PVIN2), U2.25 (PVIN2), U2.35 (PVIN1), U2.36 (PVIN1), U2.4 (PVIN3), U2.9 (PVIN4)
- net at U2.26 (SW2), U2.27 (SW2): now also JP3.2 (Pin_2), R2.1
- net at U2.3 (SW3): now also JP4.2 (Pin_2), R3.1
- net at U2.30 (PGND): now also D2.2 (A)
- net VCC3V3: now reaches U2.33 (SW1), U2.34 (SW1)
- net VCC3V3: now also U2.8 (PVIN5)
- net VCC1V0: now reaches U2.48 (EN3)
- net VCC1V0: now also JP3.1 (Pin_1), JP4.1 (Pin_1), R2.2, R3.2
- net AVCC1V8: now reaches U2.7 (VOUT5)
- new net GND: D2.1 (K)
Other:
- note added: "1A"
- note added: "2.2A"
