File: adc.kicad_sch (KiCad schematic)
At the start: 1 part, among them U6 AD9481BSUZ-250

Commit message: Uploading...
Parts:
- added C45, C46, C51, C52, C53, C54, C55, C56, C57, C58, C59, C60, C61: 0.1uF, symbol Device:C
- added C47, C48, C49, C50, C62: 10uF, symbol Device:C_Polarized_Small_US
- added C63: X, symbol Device:C
- added J10, J9: Conn_01x12, symbol Connector_Generic:Conn_01x12
- added J11, J12, J8: Conn_01x04, symbol Connector_Generic:Conn_01x04
- added R27, R28, R33, R34, R35, R36, R37, R38, R39, R40, R41, R42, R43, R44, R45, R46, R49, R50, R51, R52, R53, R54, R55, R56, R59, R60, R61, R62, R63, R64, R65, R66: 100, symbol Device:R_US
- added R29, R30, R31, R32, R47, R48, R57, R58, R67: R, symbol Device:R
- added R68, R69, R70, R71, R72, R73, R74, R75: 100, symbol Device:R
- added R76: X, symbol Device:R
- added SW1, SW2, SW3, SW4: SW_SPDT, symbol Switch:SW_SPDT
- added U12, U13: 74LVT574, symbol New_Library:74LVT574
- added U18: 74VCX86, symbol New_Library:74VCX86
Connections:
- net at U6.1 (CLK+): now also C45.2
- net DA4: now reaches U6.10 (D4A)
- net DA4: now also J9.9 (Pin_9), R53.1, R63.1
- net DA3: now reaches U6.11 (D3A)
- net DA3: now also J9.8 (Pin_8), R52.1, R62.1
- net DA2: now reaches U6.12 (D2A)
- net DA2: now also J9.7 (Pin_7), R51.1, R61.1
- net DA1: now reaches U6.13 (D1A)
- net DA1: now also J9.6 (Pin_6), R50.1, R60.1
- net DA0: now reaches U6.14 (D0A)
- net DA0: now also J9.5 (Pin_5), R49.1, R59.1
- net GND: now reaches U6.15 (DRGND_3)
- net GND: now also U6.27 (DRGND), U6.32 (AGND_3), U6.33 (SENSE), U6.35 (AGND_4), U6.37 (AGND_5), U6.4 (AGND_2), U6.40 (AGND), U6.43 (DS-), U6.44 (DS+), U6.6 (DRGND_2), C47.2, C48.2, C49.2, C50.2, C51.2, C52.2, C53.2, C54.2, C55.2, C56.2, C57.2, C58.2, C59.2, C60.2, C61.2, C62.2, C63.2, J10.1 (Pin_1), J11.1 (Pin_1), J11.3 (Pin_3), J12.1 (Pin_1), J12.3 (Pin_3), J8.3 (Pin_3), J9.1 (Pin_1), R30.2, R48.2, R58.2, SW1.3 (C), SW2.3 (C), SW3.3 (C), SW4.3 (C), U12. (VCC), U13. (VCC)
- net COUT-: now reaches U6.16 (DCO-)
- net COUT-: now also J9.2 (Pin_2), U18.12 (4A), U18.9 (3A)
- net COUT+: now reaches U6.17 (DCO+)
- net COUT+: now also J10.2 (Pin_2), U18.1 (1A), U18.4 (2A)
- net DRVDD: now reaches U6.18 (DRVDD)
- net DRVDD: now also U6.5 (DRVDD_2), C49.1, C53.1, C57.1, J11.4 (Pin_4)
- net DB0: now reaches U6.19 (D0B)
- net DB0: now also J10.5 (Pin_5), R38.1, R46.1
- net at U6.2 (CLK-): now also C46.2
- net DB1: now reaches U6.20 (D1B)
- net DB1: now also J10.6 (Pin_6), R37.1, R45.1
- net DB2: now reaches U6.21 (D2B)
- net DB2: now also J10.7 (Pin_7), R36.1, R44.1
- net DB3: now reaches U6.22 (D3B)
- net DB3: now also J10.8 (Pin_8), R35.1, R43.1
- net DB4: now reaches U6.23 (D4B)
- net DB4: now also J10.9 (Pin_9), R34.1, R42.1
- net DB5: now reaches U6.24 (D5B)
- net DB5: now also J10.10 (Pin_10), R33.1, R41.1
- net DB6: now reaches U6.25 (D6B)
- net DB6: now also J10.11 (Pin_11), R28.1, R40.1
- net DB7: now reaches U6.26 (D7B)
- net DB7: now also J10.12 (Pin_12), R27.1, R39.1
- net S1: now reaches U6.28 (S1)
- net PWDN: now reaches U6.29 (PDWN)
- net AVDD: now reaches U6.3 (AVDD_3)
- net AVDD: now also U6.30 (AVDD_2), U6.31 (AVDD_4), U6.36 (AVDD_5), U6.41 (AVDD), C48.1, C52.1, C56.1, C58.1, C61.1, J12.2 (Pin_2)
- net VREF: now reaches U6.34 (VREF)
- net VIN-: now reaches U6.38 (VIN-)
- net VIN-: now also J9.4 (Pin_4)
- net VIN+: now reaches U6.39 (VIN+)
- net VIN+: now also J10.4 (Pin_4)
- net S3: now reaches U6.42 (S3)
- net DA7: now reaches U6.7 (D7A)
- net DA7: now also J9.12 (Pin_12), R56.1, R66.1
- net DA6: now reaches U6.8 (D6A)
- net DA6: now also J9.11 (Pin_11), R55.1, R65.1
- net DA5: now reaches U6.9 (D5A)
- net DA5: now also J9.10 (Pin_10), R54.1, R64.1
- new net: R38.2, U12. (VCC)
- new net: R45.2, U12. (VCC)
- new net: R63.2, U13. (VCC)
- new net: R53.2, U13. (VCC)
- new net: R73.1, U18.8 (3Y)
- new net: R56.2, U13. (VCC)
- new net: R54.2, U13. (VCC)
- new net: R71.1, SW4.2 (B)
- new net: R71.2, U18.13 (4B)
- new net: R69.1, SW2.2 (B)
- new net: R52.2, U13. (VCC)
- new net: R72.1, U18.11 (4Y)
- new net: R66.2, U13. (VCC)
- new net: R50.2, U13. (VCC)
- new net: C45.1, R29.2, R30.1, R31.2
- new net: R39.2, U12. (VCC)
- new net: R70.1, SW3.2 (B)
- new net: R27.2, U12. (VCC)
- new net: R36.2, U12. (VCC)
- new net: R40.2, U12. (VCC)
- new net: R65.2, U13. (VCC)
- new net: R28.2, U12. (VCC)
- new net: R41.2, U12. (VCC)
- new net: R44.2, U12. (VCC)
- new net: R42.2, U12. (VCC)
- new net: R37.2, U12. (VCC)
- new net: R33.2, U12. (VCC)
- new net: R46.2, U12. (VCC)
- new net: R34.2, U12. (VCC)
- new net: R35.2, U12. (VCC)
- new net: R43.2, U12. (VCC)
- new net: R60.2, U13. (VCC)
- new net: R51.2, U13. (VCC)
- new net: R69.2, U18.5 (2B)
- new net: R68.1, SW1.2 (B)
- new net: R68.2, U18.2 (1B)
- new net: R61.2, U13. (VCC)
- new net: R49.2, U13. (VCC)
- new net: R59.2, U13. (VCC)
- new net: R62.2, U13. (VCC)
- new net: R64.2, U13. (VCC)
- new net: R55.2, U13. (VCC)
- new net: R74.1, U18.6 (2Y)
- new net: R70.2, U18.10 (3B)
- new net: R75.1, U18.3 (1Y)
- new net CLKLAT+: R47.2, R48.1, R75.2, U12. (VCC)
- new net CLKLAT-: R57.2, R58.1, R73.2, U13. (VCC)
- new net DR+: J10.3 (Pin_3), R74.2
- new net DR-: J9.3 (Pin_3), R72.2
- new net VAMP: C62.1, J8.4 (Pin_4), R76.1
- new net VAMPF: C63.1, R76.2
- new net VCTRL: C46.1, C50.1, C54.1, J12.4 (Pin_4), R29.1, R31.1, R32.1, R32.2, R67.1
- new net VDL: C47.1, C51.1, C55.1, C59.1, C60.1, J11.2 (Pin_2), R47.1, R57.1, R67.2, SW1.1 (A), SW2.1 (A), SW3.1 (A), SW4.1 (A), U12. (VCC), U13. (VCC)
Other:
- note added: "100 Ohm"
- moved on the sheet: U6

Commit message: Checked.
Other:
- moved on the sheet: J10, J8
Changed lines of the file:
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@@
 	(wire
 		(pts
-			(xy 271.78 63.5) (xy 267.97 63.5)
-		)
-		(stroke
-			(width 0)
-			(type default)
-		)
-	)
-	(wire
-		(pts
 			(xy 166.37 73.66) (xy 162.56 73.66)
 		)
@@
 	(wire
 		(pts
-			(xy 267.97 63.5) (xy 267.97 64.77)
-		)
-		(stroke
-			(width 0)
-			(type default)
-		)
-	)
-	(wire
-		(pts
 			(xy 240.03 88.9) (xy 240.03 86.36)
 		)
@@
 	(wire
 		(pts
-			(xy 267.97 64.77) (xy 266.7 64.77)
-		)
-		(stroke
-			(width 0)
-			(type default)
-		)
-	)
-	(wire
-		(pts
 			(xy 182.88 59.69) (xy 187.96 59.69)
 		)
@@
 	)
 	(label "VAMP"
-		(at 233.68 29.21 270)
+		(at 234.95 29.21 270)
 		(fields_autoplaced yes)
 		(effects
@@
 	)
 	(label "DB4"
-		(at 271.78 81.28 0)
+		(at 270.51 81.28 0)
 		(fields_autoplaced yes)
 		(effects
@@
 	)
 	(label "DB6"
-		(at 271.78 86.36 0)
+		(at 270.51 86.36 0)
 		(fields_autoplaced yes)
 		(effects
@@
 	)
 	(label "DB7"
-		(at 271.78 88.9 0)
+		(at 270.51 88.9 0)
 		(fields_autoplaced yes)
 		(effects
@@
 	)
 	(label "DR+"
-		(at 271.78 66.04 0)
+		(at 270.51 66.04 0)
 		(fields_autoplaced yes)
 		(effects
@@
 	)
 	(label "VIN+"
-		(at 271.78 68.58 0)
+		(at 270.51 68.58 0)
 		(fields_autoplaced yes)
 		(effects
@@
 	)
 	(label "DB5"
-		(at 271.78 83.82 0)
+		(at 270.51 83.82 0)
 		(fields_autoplaced yes)
 		(effects
@@
 	)
 	(label "DB2"
-		(at 271.78 76.2 0)
+		(at 270.51 76.2 0)
 		(fields_autoplaced yes)
 		(effects
@@
 	)
 	(label "GND"
-		(at 236.22 29.21 270)
+		(at 237.49 29.21 270)
 		(fields_autoplaced yes)
 		(effects
@@
 	)
 	(label "COUT+"
-		(at 266.7 64.77 0)
+		(at 270.51 63.5 0)
 		(fields_autoplaced yes)
 		(effects
@@
 	)
 	(label "GND"
-		(at 271.78 60.96 0)
+		(at 270.51 60.96 0)
 		(fields_autoplaced yes)
 		(effects
@@
 	)
 	(label "DB0"
-		(at 271.78 71.12 0)
+		(at 270.51 71.12 0)
 		(fields_autoplaced yes)
 		(effects
@@
 	)
 	(label "DB3"
-		(at 271.78 78.74 0)
+		(at 270.51 78.74 0)
 		(fields_autoplaced yes)
 		(effects
@@
 	)
 	(label "DB1"
-		(at 271.78 73.66 0)
+		(at 270.51 73.66 0)
 		(fields_autoplaced yes)
 		(effects
@@
 	(symbol
 		(lib_id "Connector_Generic:Conn_01x12")
-		(at 266.7 73.66 0)
+		(at 265.43 73.66 0)
 		(mirror y)
 		(unit 1)
@@
 		(fields_autoplaced yes)
 		(property "Reference" "J10"
-			(at 266.7 54.61 0)
+			(at 265.43 54.61 0)
 			(effects
 				(font
@@
 		)
 		(property "Value" "Conn_01x12"
-			(at 266.7 57.15 0)
+			(at 265.43 57.15 0)
 			(effects
 				(font
@@
 		)
 		(property "Footprint" ""
-			(at 266.7 73.66 0)
+			(at 265.43 73.66 0)
 			(effects
 				(font
@@
 		)
 		(property "Datasheet" "~"
-			(at 266.7 73.66 0)
+			(at 265.43 73.66 0)
 			(effects
 				(font
@@
 		)
 		(property "Description" "Generic connector, single row, 01x12, script generated (kicad-library-utils/schlib/autogen/connector/)"
-			(at 266.7 73.66 0)
+			(at 265.43 73.66 0)
 			(effects
 				(font
@@
 	(symbol
 		(lib_id "Connector_Generic:Conn_01x04")
-		(at 238.76 24.13 270)
+		(at 240.03 24.13 270)
 		(mirror x)
 		(unit 1)
@@
 		(fields_autoplaced yes)
 		(property "Reference" "J8"
-			(at 237.49 17.78 90)
+			(at 238.76 17.78 90)
 			(effects
 				(font
@@
 		)
 		(property "Value" "Conn_01x04"
-			(at 237.49 20.32 90)
+			(at 238.76 20.32 90)
 			(effects
 				(font
@@
 		)
 		(property "Footprint" ""
-			(at 238.76 24.13 0)
+			(at 240.03 24.13 0)
 			(effects
 				(font
@@
 		)
 		(property "Datasheet" "~"
-			(at 238.76 24.13 0)
+			(at 240.03 24.13 0)
 			(effects
 				(font
@@
 		)
 		(property "Description" "Generic connector, single row, 01x04, script generated (kicad-library-utils/schlib/autogen/connector/)"
-			(at 238.76 24.13 0)
+			(at 240.03 24.13 0)
 			(effects
 				(font
@@
 	)
 	(symbol
-		(lib_name "New_Library:74LVT574")
 		(lib_id "New_Library:74LVT574")
 		(at 218.44 107.95 0)
