File: ddr3.kicad_sch (KiCad schematic)
At the start: 57 parts, among them U4 MT41K128M16JT-125_K

Commit message: Checked.
Parts:
- renumbered C1 to C66, C76 to C75, C75 to C76
Connections:
- net DDRVREF: now reaches C66.2, C75.1, C76.1, U4.H1 (VREFDQ), U4.M8 (VREFCA)
- net DD3_A0 renamed DDR3_A0
- net DD3_A1 renamed DDR3_A1
- net DD3_A10 renamed DDR3_A10
- net DD3_A11 renamed DDR3_A11
- net DD3_A12 renamed DDR3_A12
- net DD3_A13 renamed DDR3_A13
- net DD3_A2 renamed DDR3_A2
- net DD3_A3 renamed DDR3_A3
- net DD3_A4 renamed DDR3_A4
- net DD3_A5 renamed DDR3_A5
- net DD3_A6 renamed DDR3_A6
- net DD3_A7 renamed DDR3_A7
- net DD3_A8 renamed DDR3_A8
- net DD3_A9 renamed DDR3_A9
- net DD3_BA0 renamed DDR3_BA0
- net DD3_BA1 renamed DDR3_BA1
- net DD3_BA2 renamed DDR3_BA2
- net DD3_CAS renamed DDR3_CAS
- net DD3_CKE0 renamed DDR3_CKE0
- net DD3_CLK0_N renamed DDR3_CLK0_N
- net DD3_CLK0_P renamed DDR3_CLK0_P
- net DD3_CS renamed DDR3_CS
- net DD3_DM0 renamed DDR3_DM0
- net DD3_DM1 renamed DDR3_DM1
- net DD3_ODT renamed DDR3_ODT
- net DD3_RAS renamed DDR3_RAS
- net DD3_WE renamed DDR3_WE
Changed lines of the file:
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@@
 	)
 	(junction
+		(at 250.19 46.99)
+		(diameter 0)
+		(color 0 0 0 0)
+	)
+	(junction
 		(at 69.85 166.37)
 		(diameter 0)
@@
 	(wire
 		(pts
-			(xy 240.03 35.56) (xy 250.19 35.56)
+			(xy 240.03 35.56) (xy 255.27 35.56)
 		)
 		(stroke
@@
 	(wire
 		(pts
+			(xy 250.19 46.99) (xy 255.27 46.99)
+		)
+		(stroke
+			(width 0)
+			(type default)
+		)
+	)
+	(wire
+		(pts
 			(xy 48.26 132.08) (xy 146.05 132.08)
 		)
@@
 		)
 	)
-	(label "DD3_BA0"
+	(label "DDR3_BA0"
 		(at 48.26 132.08 180)
 		(fields_autoplaced yes)
@@
 		)
 	)
-	(label "DD3_A0"
+	(label "DDR3_A0"
 		(at 48.26 93.98 180)
 		(fields_autoplaced yes)
@@
 		)
 	)
-	(label "DD3_CLK0_P"
+	(label "DDR3_CLK0_P"
 		(at 29.21 86.36 180)
 		(fields_autoplaced yes)
@@
 		)
 	)
-	(label "DD3_BA1"
+	(label "DDR3_BA1"
 		(at 48.26 134.62 180)
 		(fields_autoplaced yes)
@@
 		)
 	)
-	(label "DD3_WE"
+	(label "DDR3_WE"
 		(at 48.26 66.04 180)
 		(fields_autoplaced yes)
@@
 		)
 	)
-	(label "DD3_CKE0"
+	(label "DDR3_CKE0"
 		(at 48.26 83.82 180)
 		(fields_autoplaced yes)
@@
 		)
 	)
-	(label "DD3_ODT"
+	(label "DDR3_ODT"
 		(at 27.94 73.66 180)
 		(fields_autoplaced yes)
@@
 		)
 	)
-	(label "DD3_CS"
+	(label "DDR3_CS"
 		(at 48.26 68.58 180)
 		(fields_autoplaced yes)
@@
 		)
 	)
-	(label "DD3_A11"
+	(label "DDR3_A11"
 		(at 48.26 121.92 180)
 		(fields_autoplaced yes)
@@
 		)
 	)
-	(label "DD3_A6"
+	(label "DDR3_A6"
 		(at 48.26 109.22 180)
 		(fields_autoplaced yes)
@@
 		)
 	)
-	(label "DD3_A5"
+	(label "DDR3_A5"
 		(at 48.26 106.68 180)
 		(fields_autoplaced yes)
@@
 		)
 	)
-	(label "DD3_CAS"
+	(label "DDR3_CAS"
 		(at 48.26 63.5 180)
 		(fields_autoplaced yes)
@@
 	)
 	(label "DDRVCC"
-		(at 250.19 35.56 0)
+		(at 255.27 35.56 0)
 		(fields_autoplaced yes)
 		(effects
@@
 		)
 	)
-	(label "DD3_CLK0_N"
+	(label "DDR3_CLK0_N"
 		(at 35.56 88.9 180)
 		(fields_autoplaced yes)
@@
 		)
 	)
-	(label "DD3_BA2"
+	(label "DDR3_BA2"
 		(at 48.26 137.16 180)
 		(fields_autoplaced yes)
@@
 		)
 	)
-	(label "DD3_A9"
+	(label "DDR3_A9"
 		(at 48.26 116.84 180)
 		(fields_autoplaced yes)
@@
 		)
 	)
-	(label "DD3_A2"
+	(label "DDR3_A2"
 		(at 48.26 99.06 180)
 		(fields_autoplaced yes)
@@
 		)
 	)
-	(label "DD3_A13"
+	(label "DDR3_A13"
 		(at 48.26 127 180)
 		(fields_autoplaced yes)
@@
 		)
 	)
-	(label "DD3_A1"
+	(label "DDR3_A1"
 		(at 48.26 96.52 180)
 		(fields_autoplaced yes)
@@
 		)
 	)
-	(label "DD3_RAS"
+	(label "DDR3_RAS"
 		(at 48.26 60.96 180)
 		(fields_autoplaced yes)
@@
 		)
 	)
-	(label "DD3_A3"
+	(label "DDR3_A3"
 		(at 48.26 101.6 180)
 		(fields_autoplaced yes)
@@
 		)
 	)
-	(label "DD3_A7"
+	(label "DDRVREF"
+		(at 255.27 46.99 0)
+		(fields_autoplaced yes)
+		(effects
+			(font
+				(size 1.27 1.27)
+			)
+			(justify left bottom)
+		)
+	)
+	(label "DDR3_A7"
 		(at 48.26 111.76 180)
 		(fields_autoplaced yes)
@@
 		)
 	)
-	(label "DD3_DM1"
+	(label "DDR3_DM1"
 		(at 48.26 78.74 180)
 		(fields_autoplaced yes)
@@
 		)
 	)
-	(label "DD3_A10"
+	(label "DDR3_A10"
 		(at 48.26 119.38 180)
 		(fields_autoplaced yes)
@@
 		)
 	)
-	(label "DD3_A4"
+	(label "DDR3_A4"
 		(at 48.26 104.14 180)
 		(fields_autoplaced yes)
@@
 		)
 	)
-	(label "DD3_A12"
+	(label "DDR3_A12"
 		(at 48.26 124.46 180)
 		(fields_autoplaced yes)
@@
 		)
 	)
-	(label "DD3_DM0"
+	(label "DDR3_DM0"
 		(at 48.26 76.2 180)
 		(fields_autoplaced yes)
@@
 		)
 	)
-	(label "DD3_A8"
+	(label "DDR3_A8"
 		(at 48.26 114.3 180)
 		(fields_autoplaced yes)
@@
 		(on_board yes)
 		(dnp no)
-		(property "Reference" "C1"
+		(property "Reference" "C66"
 			(at 241.046 39.878 0)
 			(effects
@@
 			(project "zyma_adc_fpga_v01"
 				(path "/e72b70a1-ba8f-4002-9d33-3db12cd9fd44/5903b4aa-f29a-49a4-9430-1673a02a54f6"
-					(reference "C1")
+					(reference "C66")
 					(unit 1)
 				)
@@
 		(on_board yes)
 		(dnp no)
-		(property "Reference" "C75"
+		(property "Reference" "C76"
 			(at 241.046 52.578 0)
 			(effects
@@
 			(project ""
 				(path "/e72b70a1-ba8f-4002-9d33-3db12cd9fd44/5903b4aa-f29a-49a4-9430-1673a02a54f6"
-					(reference "C75")
+					(reference "C76")
 					(unit 1)
 				)
@@
 		(on_board yes)
 		(dnp no)
-		(property "Reference" "C76"
+		(property "Reference" "C75"
 			(at 251.206 52.578 0)
 			(effects
@@
 			(project "zyma_adc_fpga_v01"
 				(path "/e72b70a1-ba8f-4002-9d33-3db12cd9fd44/5903b4aa-f29a-49a4-9430-1673a02a54f6"
-					(reference "C76")
+					(reference "C75")
 					(unit 1)
 				)
