File: expansion.kicad_sch (KiCad schematic)
At the start: 70 parts, among them IC1 NCP380 ADJ, J1 Jack-DC, J2 Conn_01x01, Q1 PNP, Q7A NPN, Q7B NPN, Q8A NPN, Q8B NPN, U10 REF3012AIDBZT, U7 MP8756GD-Z, U8 CSD25310Q2, U9 AP2303MPTR-G1

Commit message: Uploading...
Parts:
- removed D1: LED, symbol Device:LED
Other:
- note added: "LED"
- moved on the sheet: C137, C138, C139, C140, C141, C142, C143, C144, C145, C148, C149, C158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

Commit message: Checked.
Parts:
- added D1: LED, symbol Device:LED
Connections:
- net GND: now also D1.1 (K)
- net VU: now also D1.2 (A)
Other:
- note removed: "LED"
Changed lines of the file:
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@@
 	)
 	(junction
-		(at 256.54 39.37)
-		(diameter 0)
-		(color 0 0 0 0)
-	)
-	(junction
 		(at 60.96 177.8)
 		(diameter 0)
@@
 		(at 71.12 41.91)
 	)
+	(polyline
+		(pts
+			(xy 162.052 70.866) (xy 162.052 197.866)
+		)
+		(stroke
+			(width 0)
+			(type dash)
+		)
+	)
 	(wire
 		(pts
@@
 	(wire
 		(pts
-			(xy 256.54 31.75) (xy 261.62 31.75)
+			(xy 163.83 52.07) (xy 156.21 52.07)
 		)
 		(stroke
@@
 	(wire
 		(pts
-			(xy 163.83 52.07) (xy 156.21 52.07)
+			(xy 31.75 147.32) (xy 40.64 147.32)
 		)
 		(stroke
@@
 	(wire
 		(pts
-			(xy 31.75 147.32) (xy 40.64 147.32)
+			(xy 50.8 139.7) (xy 66.04 139.7)
 		)
 		(stroke
@@
 		)
 	)
-	(wire
+	(polyline
 		(pts
-			(xy 50.8 139.7) (xy 66.04 139.7)
+			(xy 11.938 70.866) (xy 207.518 70.866)
 		)
 		(stroke
 			(width 0)
-			(type default)
+			(type dash)
 		)
 	)
@@
 	(wire
 		(pts
-			(xy 256.54 31.75) (xy 256.54 39.37)
-		)
-		(stroke
-			(width 0)
-			(type default)
-		)
-	)
-	(wire
-		(pts
 			(xy 85.09 99.06) (xy 85.09 101.6)
 		)
@@
 	(wire
 		(pts
-			(xy 80.01 86.36) (xy 80.01 71.12)
+			(xy 80.01 86.36) (xy 80.01 73.66)
 		)
 		(stroke
@@
 		)
 	)
+	(polyline
+		(pts
+			(xy 161.798 70.866) (xy 162.052 70.866)
+		)
+		(stroke
+			(width 0)
+			(type dash)
+		)
+	)
 	(wire
 		(pts
@@
 		)
 	)
+	(polyline
+		(pts
+			(xy 162.052 125.73) (xy 284.988 125.73)
+		)
+		(stroke
+			(width 0)
+			(type dash)
+		)
+	)
 	(wire
 		(pts
@@
 	(wire
 		(pts
-			(xy 26.67 71.12) (xy 26.67 86.36)
+			(xy 26.67 73.66) (xy 26.67 86.36)
 		)
 		(stroke
@@
 	(wire
 		(pts
-			(xy 251.46 39.37) (xy 245.11 39.37)
+			(xy 245.11 39.37) (xy 251.46 39.37)
 		)
 		(stroke
@@
 	(wire
 		(pts
-			(xy 261.62 39.37) (xy 256.54 39.37)
-		)
-		(stroke
-			(width 0)
-			(type default)
-		)
-	)
-	(wire
-		(pts
 			(xy 66.04 148.59) (xy 66.04 139.7)
 		)
@@
 	(wire
 		(pts
-			(xy 80.01 71.12) (xy 26.67 71.12)
+			(xy 80.01 73.66) (xy 26.67 73.66)
 		)
 		(stroke
@@
 	(wire
 		(pts
+			(xy 236.22 24.13) (xy 243.84 24.13)
+		)
+		(stroke
+			(width 0)
+			(type default)
+		)
+	)
+	(wire
+		(pts
 			(xy 97.79 139.7) (xy 68.58 139.7)
 		)
@@
 	(wire
 		(pts
-			(xy 262.89 24.13) (xy 241.3 24.13)
+			(xy 264.16 24.13) (xy 251.46 24.13)
 		)
 		(stroke
@@
 	(wire
 		(pts
-			(xy 256.54 39.37) (xy 251.46 39.37)
+			(xy 251.46 39.37) (xy 261.62 39.37)
 		)
 		(stroke
@@
 		)
 	)
+	(polyline
+		(pts
+			(xy 11.938 135.89) (xy 162.052 135.89)
+		)
+		(stroke
+			(width 0)
+			(type dash)
+		)
+	)
 	(wire
 		(pts
@@
 		)
 	)
+	(polyline
+		(pts
+			(xy 207.518 11.938) (xy 207.518 70.866)
+		)
+		(stroke
+			(width 0)
+			(type dash)
+		)
+	)
 	(wire
 		(pts
@@
 		)
 	)
-	(wire
+	(polyline
 		(pts
-			(xy 71.12 153.67) (xy 71.12 162.56)
+			(xy 207.518 70.866) (xy 284.988 70.866)
 		)
 		(stroke
 			(width 0)
-			(type default)
+			(type dash)
 		)
 	)
 	(wire
 		(pts
-			(xy 267.97 59.69) (xy 267.97 55.88)
-		)
-		(stroke
-			(width 0)
-			(type default)
-		)
-	)
-	(rectangle
-		(start 16.764 134.874)
-		(end 117.094 194.818)
-		(stroke
-			(width 0)
-			(type default)
-		)
-		(fill
-			(type none)
+			(xy 71.12 153.67) (xy 71.12 162.56)
 		)
-	)
-	(rectangle
-		(start 228.6 17.78)
-		(end 280.67 71.12)
 		(stroke
 			(width 0)
 			(type default)
 		)
-		(fill
-			(type none)
-		)
 	)
-	(rectangle
-		(start 196.85 127)
-		(end 280.67 160.02)
-		(stroke
-			(width 0)
-			(type default)
-		)
-		(fill
-			(type none)
+	(wire
+		(pts
+			(xy 267.97 59.69) (xy 267.97 55.88)
 		)
-	)
-	(rectangle
-		(start 160.274 78.232)
-		(end 279.146 126.238)
 		(stroke
 			(width 0)
 			(type default)
 		)
-		(fill
-			(type none)
-		)
 	)
 	(text "25V"
@@
 		)
 	)
-	(text "LED"
-		(exclude_from_sim no)
-		(at 238.506 24.384 0)
-		(effects
-			(font
-				(size 1.27 1.27)
-			)
-		)
-	)
 	(text "1%"
 		(exclude_from_sim no)
@@
 	)
 	(label "GND"
-		(at 261.62 31.75 0)
+		(at 251.46 39.37 0)
 		(fields_autoplaced yes)
 		(effects
@@
 		)
 	)
+	(label "GND"
+		(at 236.22 24.13 180)
+		(fields_autoplaced yes)
+		(effects
+			(font
+				(size 1.27 1.27)
+			)
+			(justify right bottom)
+		)
+	)
 	(label "XADCGND"
 		(at 208.28 148.59 180)
@@
 	)
 	(label "VU"
-		(at 262.89 24.13 0)
+		(at 264.16 24.13 0)
 		(fields_autoplaced yes)
 		(effects
@@
 					(unit 1)
 				)
+			)
+		)
+	)
+	(symbol
+		(lib_id "Device:LED")
+		(at 247.65 24.13 0)
+		(unit 1)
+		(exclude_from_sim no)
+		(in_bom yes)
+		(on_board yes)
+		(dnp no)
+		(fields_autoplaced yes)
+		(property "Reference" "D1"
+			(at 246.0625 17.78 0)
+			(effects
+				(font
+					(size 1.27 1.27)
+				)
+			)
+		)
+		(property "Value" "LED"
+			(at 246.0625 20.32 0)
+			(effects
+				(font
+					(size 1.27 1.27)
+				)
+			)
+		)
+		(property "Footprint" ""
+			(at 247.65 24.13 0)
+			(effects
+				(font
+					(size 1.27 1.27)
+				)
+				(hide yes)
+			)
+		)
+		(property "Datasheet" "~"
+			(at 247.65 24.13 0)
+			(effects
+				(font
+					(size 1.27 1.27)
+				)
+				(hide yes)
+			)
+		)
+		(property "Description" "Light emitting diode"
+			(at 247.65 24.13 0)
+			(effects
+				(font
+					(size 1.27 1.27)
+				)
+				(hide yes)
+			)
+		)
+		(pin "2"
+		)
+		(pin "1"
+		)
+		(instances
+			(project ""
+				(path "/e72b70a1-ba8f-4002-9d33-3db12cd9fd44/61aa7636-a489-4c67-86e6-82168d0668fc"
+					(reference "D1")
+					(unit 1)
+				)
