File: fpga_page3.kicad_sch (KiCad schematic)
At the start: 11 parts, among them Q4A NPN, Q4B NPN, U1 XC7S75-1FGGA484C, Y2 ASFLMB-100.000MHZ-LR-T

Commit message: Uploading...
Connections:
- net DDR3_BA0: no longer U1.Y4 (IO_L15P_T2_DQS_34)
- new net DDR3_BA2: U1.Y4 (IO_L15P_T2_DQS_34)
Other:
- moved on the sheet: U1F

Commit message: Checked.
Connections:
- net DDR3_12 renamed DDR3_A12
Changed lines of the file:
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@@
 		)
 	)
-	(label "DDR3_12"
+	(label "DDR3_A12"
 		(at 125.73 96.52 0)
 		(fields_autoplaced yes)
