File: fpga_page4.kicad_sch (KiCad schematic)
At the start: 18 parts, among them U1 XC7S75-1FGGA484C, U3 XC7S75-1FGGA484C, Y1 ASEM1-100.000MHZ-LC-T

Commit message: Uploading...
Other:
- moved on the sheet: R128

Commit message: Checked.
Other:
- note added: "No Load"
Changed lines of the file:
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@@
+		)
+	)
+	(text "No Load"
+		(exclude_from_sim no)
+		(at 143.256 159.258 0)
+		(effects
+			(font
+				(size 1 1)
+			)
+		)
+	)
+	(text "No Load"
+		(exclude_from_sim no)
+		(at 143.256 174.498 0)
+		(effects
+			(font
+				(size 1 1)
+			)
+		)
+	)
+	(text "No Load"
+		(exclude_from_sim no)
+		(at 143.256 144.018 0)
+		(effects
+			(font
+				(size 1 1)
+			)
 		)
 	)
